File: Pyramid_Shield/Pyramid_Shield.sch (KiCad schematic (older format))
At the start: 27 parts, among them P1 IR Rec, P2 Button, P3 RGB HEX, P4 GROVE, P5 IR LED, P6 Metal Shield, P7 CONN_5, P8 CONN_4, P9 CONN_5, Q1 PNP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

Commit message: New Product Importing
Parts:
- C3: value 0.1uF -> 100nF
- R3: value 820 -> 820R
- R5, R6, R7: value 330 -> 330R
- R8: value 200 -> 200R
Changed lines of the file:
@@
-EESchema Schematic File Version 2  date 7/3/2013 12:48:07
+EESchema Schematic File Version 2  date 7/10/2013 01:02:45
 LIBS:power
 LIBS:device
@@
 LIBS:Puzzlebox
 LIBS:Kicad_OSHW
+LIBS:Pyramid_Shield-cache
 EELAYER 27 0
 EELAYER END
@@
 Sheet 1 1
 Title "Puzzlebox Pyramid Shield"
-Date "27 jun 2013"
+Date "9 jul 2013"
 Rev "0.1"
 Comp "Puzzlebox Productions LLC"
@@
 P 6050 2600
 F 0 "R5" V 6130 2600 40  0000 C CNN
-F 1 "330" V 6057 2601 40  0000 C CNN
+F 1 "330R" V 6057 2601 40  0000 C CNN
 F 2 "~" V 5980 2600 30  0000 C CNN
 F 3 "~" H 6050 2600 30  0000 C CNN
@@
 P 6050 2700
 F 0 "R6" V 5950 2700 40  0000 C CNN
-F 1 "330" V 6057 2701 40  0000 C CNN
+F 1 "330R" V 6057 2701 40  0000 C CNN
 F 2 "~" V 5980 2700 30  0000 C CNN
 F 3 "~" H 6050 2700 30  0000 C CNN
@@
 P 2250 3950
 F 0 "R3" V 2330 3950 40  0000 C CNN
-F 1 "820" V 2257 3951 40  0000 C CNN
+F 1 "820R" V 2257 3951 40  0000 C CNN
 F 2 "~" V 2180 3950 30  0000 C CNN
 F 3 "~" H 2250 3950 30  0000 C CNN
@@
 P 1950 1700
 F 0 "R7" V 2030 1700 40  0000 C CNN
-F 1 "330" V 1957 1701 40  0000 C CNN
+F 1 "330R" V 1957 1701 40  0000 C CNN
 F 2 "~" V 1880 1700 30  0000 C CNN
 F 3 "~" H 1950 1700 30  0000 C CNN
@@
 P 1550 1500
 F 0 "C3" H 1550 1600 40  0000 L CNN
-F 1 "0.1uF" H 1400 1400 40  0000 L CNN
+F 1 "100nF" H 1400 1400 40  0000 L CNN
 F 2 "~" H 1588 1350 30  0000 C CNN
 F 3 "~" H 1550 1500 60  0000 C CNN
@@
 P 1650 3450
 F 0 "R8" V 1730 3450 40  0000 C CNN
-F 1 "200" V 1657 3451 40  0000 C CNN
+F 1 "200R" V 1657 3451 40  0000 C CNN
 F 2 "~" V 1580 3450 30  0000 C CNN
 F 3 "~" H 1650 3450 30  0000 C CNN
