File: RGB_HEX/RGB_HEX.sch (KiCad schematic (older format))
At the start: 44 parts, among them IC1 ATMEGA328P-M, P1 I2C, P2 FTDI, P3 ISP, Q1 NPN, Q2 NPN, Q3 NPN, Q4 NPN, Q5 NPN, Q6 NPN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

Commit message: New Product Importing
Parts:
- C2, C3, C4: value 0.1uF -> 100nF
- R1, R5: value 13k -> 1.0k 1%
- R2, R6: value 15k -> 1.2k 1%
- R3, R7: value 27k -> 2.1k 1%
Changed lines of the file:
@@
-EESchema Schematic File Version 2  date 7/1/2013 01:16:56
+EESchema Schematic File Version 2  date 7/10/2013 14:06:59
 LIBS:power
 LIBS:device
@@
 Sheet 1 1
 Title "RGB_HEX"
-Date "30 jun 2013"
+Date "10 jul 2013"
 Rev "1.3"
 Comp "Puzzlebox Productions LLC"
@@
 P 6850 4950
 F 0 "C3" H 6850 5050 40  0000 L CNN
-F 1 "0.1uF" H 6856 4865 40  0000 L CNN
+F 1 "100nF" H 6856 4865 40  0000 L CNN
 F 2 "~" H 6888 4800 30  0000 C CNN
 F 3 "~" H 6850 4950 60  0000 C CNN
@@
 P 6600 4950
 F 0 "C2" H 6600 5050 40  0000 L CNN
-F 1 "0.1uF" H 6606 4865 40  0000 L CNN
+F 1 "100nF" H 6606 4865 40  0000 L CNN
 F 2 "~" H 6638 4800 30  0000 C CNN
 F 3 "~" H 6600 4950 60  0000 C CNN
@@
 P 9350 4250
 F 0 "R1" V 9350 4050 40  0000 C CNN
-F 1 "13k" V 9357 4251 40  0000 C CNN
+F 1 "1.0k 1%" V 9357 4251 40  0000 C CNN
 F 2 "~" V 9280 4250 30  0000 C CNN
 F 3 "~" H 9350 4250 30  0000 C CNN
@@
 P 9350 4350
 F 0 "R2" V 9350 4150 40  0000 C CNN
-F 1 "15k" V 9357 4351 40  0000 C CNN
+F 1 "1.2k 1%" V 9357 4351 40  0000 C CNN
 F 2 "~" V 9280 4350 30  0000 C CNN
 F 3 "~" H 9350 4350 30  0000 C CNN
@@
 P 9350 4450
 F 0 "R3" V 9350 4250 40  0000 C CNN
-F 1 "27k" V 9357 4451 40  0000 C CNN
+F 1 "2.1k 1%" V 9357 4451 40  0000 C CNN
 F 2 "~" V 9280 4450 30  0000 C CNN
 F 3 "~" H 9350 4450 30  0000 C CNN
@@
 P 9300 6050
 F 0 "R5" V 9300 5850 40  0000 C CNN
-F 1 "13k" V 9307 6051 40  0000 C CNN
+F 1 "1.0k 1%" V 9307 6051 40  0000 C CNN
 F 2 "~" V 9230 6050 30  0000 C CNN
 F 3 "~" H 9300 6050 30  0000 C CNN
@@
 P 9300 6250
 F 0 "R6" V 9300 6050 40  0000 C CNN
-F 1 "15k" V 9307 6251 40  0000 C CNN
+F 1 "1.2k 1%" V 9307 6251 40  0000 C CNN
 F 2 "~" V 9230 6250 30  0000 C CNN
 F 3 "~" H 9300 6250 30  0000 C CNN
@@
 P 9300 6350
 F 0 "R7" V 9300 6150 40  0000 C CNN
-F 1 "27k" V 9307 6351 40  0000 C CNN
+F 1 "2.1k 1%" V 9307 6351 40  0000 C CNN
 F 2 "~" V 9230 6350 30  0000 C CNN
 F 3 "~" H 9300 6350 30  0000 C CNN
@@
 P 8850 1800
 F 0 "C4" H 8850 1900 40  0000 L CNN
-F 1 "0.1uF" H 8856 1715 40  0000 L CNN
+F 1 "100nF" H 8856 1715 40  0000 L CNN
 F 2 "~" H 8888 1650 30  0000 C CNN
 F 3 "~" H 8850 1800 60  0000 C CNN
